File: core/v0.1a/ftdi.sch (KiCad schematic (older format))
At the start: 33 parts, among them J1 Conn, P1 pkl_USB_OTG, P2 UP, P3 UP, P4 UP, P5 UP, U1 93C46B-SOT-23-6, U2 FT232H, X1 12MHz

Commit message: Changed the ftdi breakout design to use a 50mil header.
This also decreases the width of the breakout, which will allow us to
make standard complient 0.8" wide PMOD modules using the breakout board
as a basis.
Parts:
- J1: footprint Connector_PinHeader_2.54mm:PinHeader_2x10_P2.54mm_Horizontal -> pkl_samtec:FTSH-EDGE-20pin
Changed lines of the file:
@@
 F 0 "J1" H 8450 6020 50  0000 C CNN
 F 1 "Conn" H 8450 5927 50  0000 C CNN
-F 2 "Connector_PinHeader_2.54mm:PinHeader_2x10_P2.54mm_Horizontal" H 8400 5400 50  0001 C CNN
+F 2 "pkl_samtec:FTSH-EDGE-20pin" H 8400 5400 50  0001 C CNN
 F 3 "~" H 8400 5400 50  0001 C CNN
-F 4 "ANY" H 8400 5400 50  0001 C CNN "Source"
-F 5 "conn-th-01in-2-10-hdr-ra" H 100 0   50  0001 C CNN "Key"
+F 4 "conn-th-01in-2-10-hdr-ra" H 100 0   50  0001 C CNN "Key"
+F 5 "ANY" H 8400 5400 50  0001 C CNN "Source"
 	1    8400 5400
 	-1   0    0    1
