File: adapters/pmod-uart/v1.0a/ftdi-pmod-uart.sch (KiCad schematic (older format))
At the start: 2 parts, among them J1 Conn, J4 Prog

Commit message: Corrected pmod UART pinout and added INT/RST pins.
Parts:
- J4: value Prog -> PMOD; footprint Connector_PinSocket_2.54mm:PinSocket_1x06_P2.54mm_Vertical -> Connector_PinHeader_2.54mm:PinHeader_2x06_P2.54mm_Horizontal; symbol Connector_Generic:Conn_01x06 -> Connector_Generic:Conn_02x06_Odd_Even
Connections:
- net ACBUS1: now also J4.4 (Pin_4)
- net ACBUS2: now also J4.2 (Pin_2)
- net GND: now also J4.10 (Pin_10), J4.9 (Pin_9); no longer J4.6 (Pin_6)
- net TXD: now also J4.5 (Pin_5); no longer J4.4 (Pin_4)
- net ~CTS: now also J4.7 (Pin_7); no longer J4.1 (Pin_1)
- net ~RTS: now also J4.1 (Pin_1); no longer J4.2 (Pin_2)
- net ~WRSAV renamed ~PWRSAV
- no-connect marks 1 -> 4
Other:
- note added: "PMOD Interface Type 4 (UART)"
- note removed: "~WRSAV"
Changed lines of the file:
@@
 EESchema Schematic File Version 4
-LIBS:ftdi-pmod-spi-cache
+LIBS:ftdi-pmod-uart-cache
 EELAYER 26 0
 EELAYER END
@@
 ACBUS6
 Text Label 3500 2100 0    50   ~ 0
-~WRSAV
+~PWRSAV
 Text Label 2600 2200 2    50   ~ 0
 ACBUS8
@@
 ACBUS8
 Text Notes 2450 5150 0    50   ~ 0
-~WRSAV
+~PWRSAV
 Text Notes 2450 5050 0    50   ~ 0
 ACBUS6
@@
 	2700 1300 2700 2400
 $Comp
-L Connector_Generic:Conn_01x06 J4
+L Connector_Generic:Conn_02x06_Odd_Even J4
 U 1 1 5AB98614
 P 5000 1700
 F 0 "J4" H 4950 2000 50  0000 L CNN
-F 1 "Prog" H 4850 2100 50  0000 L CNN
-F 2 "Connector_PinSocket_2.54mm:PinSocket_1x06_P2.54mm_Vertical" H 5000 1700 50  0001 C CNN
+F 1 "PMOD" H 4850 2100 50  0000 L CNN
+F 2 "Connector_PinHeader_2.54mm:PinHeader_2x06_P2.54mm_Horizontal" H 5000 1700 50  0001 C CNN
 F 3 "~" H 5000 1700 50  0001 C CNN
 F 4 "ANY" H 5000 1700 50  0001 C CNN "Source"
@@
 	4800 1800 4600 1800
 Wire Wire Line
-	4800 2000 4700 2000
+	4800 1900 4700 1900
+Text Label 4600 1500 2    50   ~ 0
+~RTS
 Text Label 4600 1600 2    50   ~ 0
-~RTS
-Text Label 4600 1700 2    50   ~ 0
 RXD
 Wire Wire Line
-	4700 2000 4700 2100
+	4700 1900 4700 2100
 $Comp
 L power:GND #PWR0103
@@
 	1    0    0    -1
 $EndComp
+Text Label 4600 1700 2    50   ~ 0
+TXD
+NoConn ~ 4800 2000
 Text Label 4600 1800 2    50   ~ 0
-TXD
-NoConn ~ 4800 1900
-Text Label 4600 1500 2    50   ~ 0
 ~CTS
+Text Notes 4450 1150 0    50   ~ 0
+PMOD Interface Type 4 (UART)
+Wire Wire Line
+	5300 1500 5400 1500
+Wire Wire Line
+	5300 1600 5400 1600
+Wire Wire Line
+	5300 1900 5400 1900
+Wire Wire Line
+	5400 1900 5400 2100
+$Comp
+L power:GND #PWR0104
+U 1 1 5AAB5F9F
+P 5400 2100
+F 0 "#PWR0104" H 5400 1850 50  0001 C CNN
+F 1 "GND" H 5405 1924 50  0000 C CNN
+F 2 "" H 5400 2100 50  0001 C CNN
+F 3 "" H 5400 2100 50  0001 C CNN
+	1    5400 2100
+	1    0    0    -1
+$EndComp
+NoConn ~ 5300 1700
+NoConn ~ 5300 1800
+NoConn ~ 5300 2000
+Text Label 5400 1600 0    50   ~ 0
+ACBUS1
+Text Label 5400 1500 0    50   ~ 0
+ACBUS2
 $EndSCHEMATC
