File: adapters/100mil/v1.0a/ftdi-100mil.sch (KiCad schematic (older format))
At the start: 2 parts, among them J1 Conn, J2 Conn

Commit message: A bunch of minor fixes.
* PWRSAV instead of WRSAV in signal table.
* 0.05 solder stop opening instead of 0.2
* Better copper fill parameters.
Other:
- note removed: "~WRSAV"
Changed lines of the file:
@@
 ACBUS8
 Text Notes 2450 5150 0    50   ~ 0
-~WRSAV
+~PWRSAV
 Text Notes 2450 5050 0    50   ~ 0
 ACBUS6
