File: adapters/bitsy-prog/v1.0a/ftdi-bitsy-prog.kicad_pcb (KiCad board)
At the start: 2 copper layers, 19 x 22 mm, 4 parts, among them J1 Conn, J2 CS, J3 GND, J4 Prog

Commit message: A bunch of minor fixes.
* PWRSAV instead of WRSAV in signal table.
* 0.05 solder stop opening instead of 0.2
* Better copper fill parameters.
Other:
- rule pad_to_mask_clearance: 0.2 -> 0.05
Changed lines of the file:
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@@
-(kicad_pcb (version 20171130) (host pcbnew 5.0.0-rc2-dev-unknown-d64c89d~62~ubuntu16.04.1)
+(kicad_pcb (version 20171130) (host pcbnew 5.0.0-rc2-dev-unknown-c6ef0d5~62~ubuntu16.04.1)
   (general
     (thickness 0.8)
@@
     (last_trace_width 0.25)
     (trace_clearance 0.2)
-    (zone_clearance 0.508)
+    (zone_clearance 0.25)
     (zone_45_only yes)
     (trace_min 0.2)
@@
     (pad_size 1.524 1.524)
     (pad_drill 0.762)
-    (pad_to_mask_clearance 0.2)
+    (pad_to_mask_clearance 0.05)
     (aux_axis_origin 0 0)
     (grid_origin 47 44)
@@
   (segment (start 46.93 42.8) (end 47 42.73) (width 0.25) (layer F.Cu) (net 10))
   (zone (net 1) (net_name GND) (layer F.Cu) (hatch edge 0.508)
-    (connect_pads (clearance 0.508))
-    (min_thickness 0.254)
-    (fill yes (arc_segments 16) (thermal_gap 0.508) (thermal_bridge_width 0.508))
+    (connect_pads (clearance 0.25))
+    (min_thickness 0.25)
+    (fill yes (arc_segments 16) (thermal_gap 0.25) (thermal_bridge_width 0.26))
     (polygon
       (pts
@@
   )
   (zone (net 1) (net_name GND) (layer B.Cu) (hatch edge 0.508)
-    (connect_pads (clearance 0.508))
-    (min_thickness 0.254)
-    (fill yes (arc_segments 16) (thermal_gap 0.508) (thermal_bridge_width 0.508))
+    (connect_pads (clearance 0.25))
+    (min_thickness 0.25)
+    (fill yes (arc_segments 16) (thermal_gap 0.25) (thermal_bridge_width 0.26))
     (polygon
       (pts
