File: core/v1.0a/ftdi.kicad_pcb (KiCad board)
At the start: 2 copper layers, 32 x 20 mm, 35 parts, among them J1 Conn, P1 pkl_USB_OTG, P2 UP, P3 UP, P4 UP, P5 UP, U1 93C46B-SOT-23-6, U2 FT232H, X1 12MHz

Commit message: Improved legend of the FT232 USBtoX Multitool Breakout.
Other:
- board text added: "FT232H USBtoX Multitool Breakout V1.0a"
- board text removed: "FT232H Breakout V1.0a"
Changed lines of the file:
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@@
 (kicad_pcb (version 20171130) (host pcbnew 5.0.0-rc2-dev-unknown-c6ef0d5~62~ubuntu16.04.1)
   (general
-    (thickness 1.6)
+    (thickness 0.8)
     (drawings 44)
     (tracks 345)
@@
     (effects (font (size 0.75 0.75) (thickness 0.1875)) (justify left mirror))
   )
-  (gr_text "FT232H Breakout\nV1.0a" (at 49.7 47.6 270) (layer B.SilkS)
+  (gr_text "FT232H USBtoX\nMultitool Breakout\nV1.0a" (at 49.7 47.6 270) (layer B.SilkS)
     (effects (font (size 1 1) (thickness 0.25)) (justify mirror))
   )
@@
     (effects (font (size 0.9 0.9) (thickness 0.225)) (justify right))
   )
-  (gr_text "FT232H Breakout V1.0a" (at 31.3 56.6) (layer F.SilkS)
+  (gr_text "FT232H USBtoX\nMultitool Breakout V1.0a" (at 30.8 55.6) (layer F.SilkS)
     (effects (font (size 1 1) (thickness 0.25)) (justify left))
   )
